File: PCB/PCB_new/LAUNCHXL-F28379D_Headers.sch (KiCad schematic (older format))
At the start: 12 parts, among them J1 SSW-110-02-G-S, J2 SSW-110-02-G-S, J3 SSW-110-02-G-S, J4 SSW-110-02-G-S, J5 SSW-110-02-G-S, J6 SSW-110-02-G-S, J7 SSW-110-02-G-S, J8 SSW-110-02-G-S

Commit message: updated schematic and packages (need to verify many packages)
Parts:
- C2, C3, C4, C5: symbol PCB_HEADERS_2020-rescue:C-PCB_Sch-eagle-import -> PCB_2020:C-PCB_Sch-eagle-import
- J1, J2, J3, J4, J5, J6, J7, J8: symbol PCB_HEADERS_2020-rescue:SSW-110-02-G-S-PCB_Sch-eagle-import -> PCB_2020:SSW-110-02-G-S-PCB_Sch-eagle-import
Connections:
- net labels added: GND-PCB_Sch-eagle-import
- wire segments 97 -> 98

Commit message: cleaned up breakout and headers files
Parts:
- removed J1, J2, J3, J5, J6, J7, J8: SSW-110-02-G-S, PCB_Sch:SSW-110-02-G-S, symbol PCB_2020:SSW-110-02-G-S-PCB_Sch-eagle-import
- removed unit 1 of J4
- removed unit 3 of J4
- removed unit 2 of J4
- removed unit 5 of J4
- removed unit 4 of J4
- removed unit 7 of J4
- removed unit 6 of J4
- removed unit 9 of J4
- removed unit 8 of J4
- added J?: TI_TRR, Connector_Samtec_HLE_THT:Samtec_HLE-110-02-xx-DV-TE_2x10_P2.54mm_Horizontal, symbol Connector:Conn_01x10_Female
- added J?: TI_TRL, Connector_Samtec_HLE_THT:Samtec_HLE-110-02-xx-DV-TE_2x10_P2.54mm_Horizontal, symbol Connector:Conn_01x10_Female
- added J?: TI_TLR, Connector_Samtec_HLE_THT:Samtec_HLE-110-02-xx-DV-TE_2x10_P2.54mm_Horizontal, symbol Connector:Conn_01x10_Female
- added J?: TI_TLL, Connector_Samtec_HLE_THT:Samtec_HLE-110-02-xx-DV-TE_2x10_P2.54mm_Horizontal, symbol Connector:Conn_01x10_Female
- added J?: TI_BLL, Connector_Samtec_HLE_THT:Samtec_HLE-110-02-xx-DV-TE_2x10_P2.54mm_Horizontal, symbol Connector:Conn_01x10_Female
- added J?: TI_BLR, Connector_Samtec_HLE_THT:Samtec_HLE-110-02-xx-DV-TE_2x10_P2.54mm_Horizontal, symbol Connector:Conn_01x10_Female
- added J?: TI_BRL, Connector_Samtec_HLE_THT:Samtec_HLE-110-02-xx-DV-TE_2x10_P2.54mm_Horizontal, symbol Connector:Conn_01x10_Female
- added J?: TI_BRR, Connector_Samtec_HLE_THT:Samtec_HLE-110-02-xx-DV-TE_2x10_P2.54mm_Horizontal, symbol Connector:Conn_01x10_Female
- C2, C3, C4, C5: symbol PCB_2020:C-PCB_Sch-eagle-import -> Device:C
- J4: footprint PCB_Sch:SSW-110-02-G-S -> Connector_Samtec_HLE_THT:Samtec_HLE-110-02-xx-DV-TE_2x10_P2.54mm_Horizontal
Connections:
- net +3V3: now also J?.1 (Pin_1), J?.1 (Pin_1)
- net +5V: now also J?.1 (Pin_1), J?.1 (Pin_1)
- net ADCA0: now also J?.10 (Pin_10)
- net ADCIN1: now also J?.3 (Pin_3)
- net ADCIN15: now also J?.3 (Pin_3)
- net ADCINA2: now also J?.9 (Pin_9)
- net ADCINA3: now also J?.6 (Pin_6)
- net ADCINA4: now also J?.9 (Pin_9)
- net ADCINA5: now also J?.6 (Pin_6)
- net ADCINB2: now also J?.8 (Pin_8)
- net ADCINB3: now also J?.5 (Pin_5)
- net ADCINB4: now also J?.8 (Pin_8)
- net ADCINB5: now also J?.5 (Pin_5)
- net ADCINC2: now also J?.7 (Pin_7)
- net ADCINC3: now also J?.4 (Pin_4)
- net ADCINC4: now also J?.7 (Pin_7)
- net ADCINC5: now also J?.4 (Pin_4)
- net EN+_CTL: now also J?.7 (Pin_7)
- net FEATHER_RESET: now also J?.2 (Pin_2)
- net FS1_CTL: now also J?.1 (Pin_1)
- net FWD_CTL: now also J?.2 (Pin_2)
- net GND: now also J?.1 (Pin_1), J?.1 (Pin_1), J?.2 (Pin_2), J?.2 (Pin_2)
- net GPIO111: now also J?.6 (Pin_6)
- net GPIO22: now also J?.8 (Pin_8)
- net GPIO32: now also J?.2 (Pin_2)
- net GPIO67: now also J?.5 (Pin_5)
- net GPIO94: now also J?.6 (Pin_6)
- net I2CSCLB: now also J?.9 (Pin_9)
- net I2CSDAB: now also J?.10 (Pin_10)
- net INPUT_A+_CTL: now also J?.8 (Pin_8)
- net KILL_SIGNAL: now also J?.5 (Pin_5)
- net MC_HLFB+: now also J?.7 (Pin_7)
- net MC_U: now also J?.4 (Pin_4)
- net MC_V: now also J?.5 (Pin_5)
- net MC_W: now also J?.6 (Pin_6)
- net RESET: now also J?.5 (Pin_5), J?.5 (Pin_5)
- net REV_CTL: now also J?.3 (Pin_3)
- net SCIB_RX: now also J?.3 (Pin_3)
- net SCIB_TX: now also J?.4 (Pin_4)
- net THROTTLE_DAC: now also J?.10 (Pin_10)
- net TI_PWM: now also J?.1 (Pin_1); no longer J4.10 (1)
- new net GPIO1-PWMOUT1B: J?.2 (Pin_2)
- new net GPIO104-I2CSDAA-J1: J?.10 (Pin_10)
- new net GPIO105-I2SSCLA-J1: J?.9 (Pin_9)
- new net GPIO122-SD1D1: J?.4 (Pin_4)
- new net GPIO123-SD1CLK1: J?.3 (Pin_3)
- new net GPIO124-SD1D2: J?.8 (Pin_8)
- new net GPIO125-SD1CLK2: J?.9 (Pin_9)
- new net GPIO130-SD2D1: J?.4 (Pin_4)
- new net GPIO131-SD2CLK1: J?.3 (Pin_3)
- new net GPIO139-SCICRX(->MCU): J?.3 (Pin_3)
- new net GPIO15-OPXBAR4: J?.8 (Pin_8)
- new net GPIO2-PWMOUT2A: J?.3 (Pin_3)
- new net GPIO25-OPXBAR2: J?.10 (Pin_10)
- new net GPIO26-SD2D2: J?.8 (Pin_8)
- new net GPIO27-SD2CLK2: J?.9 (Pin_9)
- new net GPIO29-OPXBAR6: J?.10 (Pin_10)
- new net GPIO3-PWMOUT2B: J?.4 (Pin_4)
- new net GPIO4-PWMOUT3A: J?.5 (Pin_5)
- new net GPIO5-PWMOUT3B: J?.6 (Pin_6)
- new net GPIO52-J5: J?.8 (Pin_8)
- new net GPIO56-SCICTX(<-MCU): J?.4 (Pin_4)
- new net GPIO58-SPIAMOSI: J?.6 (Pin_6)
- new net GPIO59-SPIAMISO: J?.7 (Pin_7)
- new net GPIO60-SPICLKA: J?.7 (Pin_7)
- new net GPIO61-SPIACS: J?.2 (Pin_2)
- new net GPIO63-SPIBMOSI: J?.6 (Pin_6)
- new net GPIO64-SPIBMISO: J?.7 (Pin_7)
- new net GPIO65-SPIBCLK: J?.7 (Pin_7)
- new net GPIO66-SPIBCS: J?.2 (Pin_2)
- new net PWM-BASED-DAC1: J?.9 (Pin_9)
- new net PWM-BASED-DAC2: J?.10 (Pin_10)
- new net PWM-BASED-DAC3: J?.9 (Pin_9)
- new net PWM-BASED-DAC4: J?.10 (Pin_10)
Other:
- note added: "PCB_Sch:SSW-110-02-G-S"
- moved on the sheet: J4J

Commit message: cleaned up .lib files
Parts:
- J4: symbol PCB_2020:SSW-110-02-G-S-PCB_Sch-eagle-import -> PCB_2020:SSW-110-02-G-S
Changed lines of the file:
@@
 SCIB_TX
 $Comp
-L PCB_2020:SSW-110-02-G-S-PCB_Sch-eagle-import J4
+L PCB_2020:SSW-110-02-G-S J4
 U 10 1 5FA1416F
 P 10900 3100

Commit message: added no connection indicators
Parts:
- gave numbers to parts that had none: 8
Connections:
- wire segments 38 -> 78
- no-connect marks 0 -> 55
Other:
- moved on the sheet: J2, J9

Commit message: changed components footprints to Drivetrain.pretty
Parts:
- removed J4: SSW-110-02-G-S, Connector_Samtec_HLE_THT:Samtec_HLE-110-02-xx-DV-TE_2x10_P2.54mm_Horizontal, symbol PCB_2020:SSW-110-02-G-S
- C2, C3, C4, C5: footprint PCB_Sch:C0805 -> Capacitor_SMD:C_0805_2012Metric_Pad1.15x1.40mm_HandSolder
- J1, J2, J3, J5, J6, J7, J8, J9: footprint Connector_Samtec_HLE_THT:Samtec_HLE-110-02-xx-DV-TE_2x10_P2.54mm_Horizontal -> Drivetrain_control:SSW-110-02-G-S
Other:
- note removed: "PCB_Sch:SSW-110-02-G-S"
Changed lines of the file:
@@
 SCIB_TX
-$Comp
-L PCB_2020:SSW-110-02-G-S J4
-U 10 1 5FA1416F
-P 10900 3100
-AR Path="/5FA1416F" Ref="J4"  Part="10"
-AR Path="/5DF27589/5FA1416F" Ref="J4"  Part="10"
-F 0 "J4" H 10780 3130 51  0000 R TNN
-F 1 "SSW-110-02-G-S" H 10800 3200 59  0001 L BNN
-F 2 "Connector_Samtec_HLE_THT:Samtec_HLE-110-02-xx-DV-TE_2x10_P2.54mm_Horizontal" H 10900 3100 50  0001 C CNN
-F 3 "" H 10900 3100 50  0001 C CNN
-	10   10900 3100
-	-1   0    0    1
-$EndComp
 $Comp
 L Device:C C2
@@
 F 0 "C2" H 3360 6115 59  0000 L BNN
 F 1 "0.1uF" H 3360 5915 59  0000 L BNN
-F 2 "PCB_Sch:C0805" H 3300 6100 50  0001 C CNN
+F 2 "Capacitor_SMD:C_0805_2012Metric_Pad1.15x1.40mm_HandSolder" H 3300 6100 50  0001 C CNN
 F 3 "" H 3300 6100 50  0001 C CNN
 	1    3300 6100
@@
 F 0 "C3" H 3860 6115 59  0000 L BNN
 F 1 "0.1uF" H 3860 5915 59  0000 L BNN
-F 2 "PCB_Sch:C0805" H 3800 6100 50  0001 C CNN
+F 2 "Capacitor_SMD:C_0805_2012Metric_Pad1.15x1.40mm_HandSolder" H 3800 6100 50  0001 C CNN
 F 3 "" H 3800 6100 50  0001 C CNN
 	1    3800 6100
@@
 F 0 "C4" H 4360 6115 59  0000 L BNN
 F 1 "0.1uF" H 4360 5915 59  0000 L BNN
-F 2 "PCB_Sch:C0805" H 4300 6100 50  0001 C CNN
+F 2 "Capacitor_SMD:C_0805_2012Metric_Pad1.15x1.40mm_HandSolder" H 4300 6100 50  0001 C CNN
 F 3 "" H 4300 6100 50  0001 C CNN
 	1    4300 6100
@@
 F 0 "C5" H 4860 6115 59  0000 L BNN
 F 1 "0.1uF" H 4860 5915 59  0000 L BNN
-F 2 "PCB_Sch:C0805" H 4800 6100 50  0001 C CNN
+F 2 "Capacitor_SMD:C_0805_2012Metric_Pad1.15x1.40mm_HandSolder" H 4800 6100 50  0001 C CNN
 F 3 "" H 4800 6100 50  0001 C CNN
 	1    4800 6100
@@
 Text Label 9200 1300 2    39   ~ 0
 GPIO61-SPIACS
-Text Notes 10150 2700 0    50   ~ 0
-PCB_Sch:SSW-110-02-G-S
 $Comp
 L Connector:Conn_01x10_Female J8
@@
 F 0 "J8" H 9428 1576 50  0000 L CNN
 F 1 "TI_TRR" H 9428 1485 50  0000 L CNN
-F 2 "Connector_Samtec_HLE_THT:Samtec_HLE-110-02-xx-DV-TE_2x10_P2.54mm_Horizontal" H 9400 1600 50  0001 C CNN
+F 2 "Drivetrain_control:SSW-110-02-G-S" H 9400 1600 50  0001 C CNN
 F 3 "~" H 9400 1600 50  0001 C CNN
 	1    9400 1600
@@
 F 0 "J7" H 8328 1576 50  0000 L CNN
 F 1 "TI_TRL" H 8328 1485 50  0000 L CNN
-F 2 "Connector_Samtec_HLE_THT:Samtec_HLE-110-02-xx-DV-TE_2x10_P2.54mm_Horizontal" H 8300 1600 50  0001 C CNN
+F 2 "Drivetrain_control:SSW-110-02-G-S" H 8300 1600 50  0001 C CNN
 F 3 "~" H 8300 1600 50  0001 C CNN
 	1    8300 1600
@@
 F 0 "J5" H 3878 1526 50  0000 L CNN
 F 1 "TI_TLR" H 3878 1435 50  0000 L CNN
-F 2 "Connector_Samtec_HLE_THT:Samtec_HLE-110-02-xx-DV-TE_2x10_P2.54mm_Horizontal" H 3850 1550 50  0001 C CNN
+F 2 "Drivetrain_control:SSW-110-02-G-S" H 3850 1550 50  0001 C CNN
 F 3 "~" H 3850 1550 50  0001 C CNN
 	1    3850 1550
@@
 F 0 "J1" H 2578 1526 50  0000 L CNN
 F 1 "TI_TLL" H 2578 1435 50  0000 L CNN
-F 2 "Connector_Samtec_HLE_THT:Samtec_HLE-110-02-xx-DV-TE_2x10_P2.54mm_Horizontal" H 2550 1550 50  0001 C CNN
+F 2 "Drivetrain_control:SSW-110-02-G-S" H 2550 1550 50  0001 C CNN
 F 3 "~" H 2550 1550 50  0001 C CNN
 	1    2550 1550
@@
 F 0 "J2" H 2428 3826 50  0000 L CNN
 F 1 "TI_BLL" H 2428 3735 50  0000 L CNN
-F 2 "Connector_Samtec_HLE_THT:Samtec_HLE-110-02-xx-DV-TE_2x10_P2.54mm_Horizontal" H 2400 3850 50  0001 C CNN
+F 2 "Drivetrain_control:SSW-110-02-G-S" H 2400 3850 50  0001 C CNN
 F 3 "~" H 2400 3850 50  0001 C CNN
 	1    2400 3850
@@
 F 0 "J3" H 3828 3826 50  0000 L CNN
 F 1 "TI_BLR" H 3828 3735 50  0000 L CNN
-F 2 "Connector_Samtec_HLE_THT:Samtec_HLE-110-02-xx-DV-TE_2x10_P2.54mm_Horizontal" H 3800 3850 50  0001 C CNN
+F 2 "Drivetrain_control:SSW-110-02-G-S" H 3800 3850 50  0001 C CNN
 F 3 "~" H 3800 3850 50  0001 C CNN
 	1    3800 3850
@@
 F 0 "J6" H 8228 3776 50  0000 L CNN
 F 1 "TI_BRL" H 8228 3685 50  0000 L CNN
-F 2 "Connector_Samtec_HLE_THT:Samtec_HLE-110-02-xx-DV-TE_2x10_P2.54mm_Horizontal" H 8200 3800 50  0001 C CNN
+F 2 "Drivetrain_control:SSW-110-02-G-S" H 8200 3800 50  0001 C CNN
 F 3 "~" H 8200 3800 50  0001 C CNN
 	1    8200 3800
@@
 F 0 "J9" H 9528 3776 50  0000 L CNN
 F 1 "TI_BRR" H 9528 3685 50  0000 L CNN
-F 2 "Connector_Samtec_HLE_THT:Samtec_HLE-110-02-xx-DV-TE_2x10_P2.54mm_Horizontal" H 9500 3800 50  0001 C CNN
+F 2 "Drivetrain_control:SSW-110-02-G-S" H 9500 3800 50  0001 C CNN
 F 3 "~" H 9500 3800 50  0001 C CNN
 	1    9500 3800

Commit message: Created TI schematic and Footprint
Parts:
- removed J1: TI_TLL, Drivetrain_control:SSW-110-02-G-S, symbol Connector:Conn_01x10_Female
- removed J2: TI_BLL, Drivetrain_control:SSW-110-02-G-S, symbol Connector:Conn_01x10_Female
- removed J3: TI_BLR, Drivetrain_control:SSW-110-02-G-S, symbol Connector:Conn_01x10_Female
- removed J5: TI_TLR, Drivetrain_control:SSW-110-02-G-S, symbol Connector:Conn_01x10_Female
- removed J6: TI_BRL, Drivetrain_control:SSW-110-02-G-S, symbol Connector:Conn_01x10_Female
- removed J7: TI_TRL, Drivetrain_control:SSW-110-02-G-S, symbol Connector:Conn_01x10_Female
- removed J8: TI_TRR, Drivetrain_control:SSW-110-02-G-S, symbol Connector:Conn_01x10_Female
- removed J9: TI_BRR, Drivetrain_control:SSW-110-02-G-S, symbol Connector:Conn_01x10_Female
- added U1: TI_CONN, Drivetrain_control:TI_Footprint, symbol PCB_2020:TI_CONN

Commit message: added braking signals
Connections:
- net labels added: Brake_PWM_1, Brake_PWM_2
- net labels removed: GPIO4-PWMOUT3A, GPIO5-PWMOUT3B
- no-connect marks 55 -> 53
Changed lines of the file:
@@
 Text Label 8300 2150 2    39   ~ 0
 GPIO2-PWMOUT2A
-Text Label 8300 2350 2    39   ~ 0
-GPIO4-PWMOUT3A
 Text GLabel 8300 2650 0    39   Input ~ 0
 INPUT_A+_CTL
@@
 Text Label 8300 2050 2    39   ~ 0
 GPIO1-PWMOUT1B
-Text Label 8300 2450 2    39   ~ 0
-GPIO5-PWMOUT3B
 Text GLabel 9800 1950 2    39   BiDi ~ 0
 GND
@@
 NoConn ~ 8300 2150
 NoConn ~ 8300 2250
-NoConn ~ 8300 2350
-NoConn ~ 8300 2450
 NoConn ~ 8300 2750
 NoConn ~ 8300 2850
@@
 Text Label 4950 3750 2    39   ~ 0
 GPIO56-SCICTX(<-MCU)
+Text GLabel 4950 3450 0    39   BiDi ~ 0
++3V3
+Wire Wire Line
+	3300 6500 3800 6500
+Text GLabel 8300 2450 0    39   Output ~ 0
+Brake_PWM_2
+Text GLabel 8300 2350 0    39   Output ~ 0
+Brake_PWM_1
 Text GLabel 4950 3550 0    39   BiDi ~ 0
 FEATHER_RESET
-Text GLabel 4950 3450 0    39   BiDi ~ 0
-+3V3
-Wire Wire Line
-	3300 6500 3800 6500
 $EndSCHEMATC

Commit message: updated component values
Connections:
- net labels removed: FEATHER_RESET, I2CSCLB, I2CSDAB, KILL_SIGNAL, MC_U, MC_V, MC_W
- no-connect marks 53 -> 58
Changed lines of the file:
@@
 Text GLabel 6550 3550 2    39   BiDi ~ 0
-GND
-Text GLabel 10000 3450 2    39   BiDi ~ 0
 GND
 Wire Wire Line
@@
 Text GLabel 8150 4050 0    39   BiDi ~ 0
 MC_HLFB+
-Text GLabel 8150 3950 0    39   BiDi ~ 0
-MC_W
-Text GLabel 8150 3850 0    39   BiDi ~ 0
-MC_V
-Text GLabel 8150 3750 0    39   BiDi ~ 0
-MC_U
 Text GLabel 8150 3650 0    39   BiDi ~ 0
 REV_CTL
@@
 NoConn ~ 9850 3650
 NoConn ~ 9850 3550
-NoConn ~ 9850 3850
-NoConn ~ 9800 2350
 NoConn ~ 6400 2150
 NoConn ~ 6400 2250
@@
 	10000 3550 9850 3550
 Wire Wire Line
-	10000 3450 9850 3450
-Wire Wire Line
 	10000 3850 9850 3850
 $Comp
@@
 Text Label 4950 3650 2    39   ~ 0
 GPIO139-SCICRX(->MCU)
-Text GLabel 4950 4350 0    39   BiDi ~ 0
-I2CSDAB
-Text GLabel 4950 4250 0    39   BiDi ~ 0
-I2CSCLB
 Text Label 4950 4150 2    39   ~ 0
 GPIO52-J5
@@
 Text Label 4950 3950 2    39   ~ 0
 GPIO94
-Text GLabel 4950 3850 0    39   BiDi ~ 0
-KILL_SIGNAL
 Text Label 4950 3750 2    39   ~ 0
 GPIO56-SCICTX(<-MCU)
@@
 Text GLabel 8300 2350 0    39   Output ~ 0
 Brake_PWM_1
-Text GLabel 4950 3550 0    39   BiDi ~ 0
-FEATHER_RESET
+Wire Wire Line
+	10000 3450 9850 3450
+Text GLabel 10000 3450 2    39   BiDi ~ 0
+GND
+NoConn ~ 8150 3750
+NoConn ~ 8150 3850
+NoConn ~ 8150 3950
+NoConn ~ 4950 3550
+NoConn ~ 4950 3850
+NoConn ~ 4950 4250
+NoConn ~ 4950 4350
 $EndSCHEMATC
