File: PCB/PCB_new/LAUNCHXL-F28379D_Headers.sch (KiCad schematic (older format))
At the start: 9 parts, among them U1 AMP_DUE_SCH

Commit message: added arduino units a, b, c, d, e
Parts:
- removed U1: AMP_DUE_SCH, DUE Footprint:Arduino DUE, symbol PCB_2020:AMP_DUE_SCH
- added U1, U2: AMP_DUE_SCH, DUE Footprint:Arduino DUE, symbol PCB_2020:AMP_DUE_SCH
Connections:
- net +5V: now also U2.66 (5V)
- net Brake_PWM_1: now also U1.3
- net Brake_PWM_2: now also U1.4
- net EN+_CTL: now also U1.31
- net FS1_CTL: now also U1.23
- net FWD_CTL: now also U1.27
- net GND: now also U2.41 (GND)
- net INPUT_A+_CTL: now also U1.33
- net KS1_CTL: now also U1.25
- net REV_CTL: now also U1.29
- net STEERING: now also U1.2
- net THROTTLE: now also U1.1 (DAC0)
- new net +12V: U2.24 (VIN)
- no-connect marks 0 -> 37
Changed lines of the file:
@@
 Connection ~ 3800 6500
 Connection ~ 4100 6500
-Wire Wire Line
-	10000 3550 10100 3550
-Text GLabel 10100 3550 2    39   BiDi ~ 0
+Text GLabel 11350 3250 2    39   BiDi ~ 0
 SCIB_RX
 $Comp
@@
 	1    0    0    -1
 $EndComp
+Text Notes 3700 7200 0    59   ~ 0
+Decoupling Caps
+$Comp
+L power:GND #GND3
+U 1 1 E2B99DEF
+P 4100 6700
+AR Path="/E2B99DEF" Ref="#GND3"  Part="1"
+AR Path="/5DF27589/E2B99DEF" Ref="#GND03"  Part="1"
+F 0 "#GND03" H 4100 6700 50  0001 C CNN
+F 1 "GND" H 4000 6500 59  0000 L BNN
+F 2 "" H 4100 6700 50  0001 C CNN
+F 3 "" H 4100 6700 50  0001 C CNN
+	1    4100 6700
+	1    0    0    -1
+$EndComp
+Wire Wire Line
+	3300 5900 3300 5950
+Wire Wire Line
+	3300 6250 3300 6500
+Wire Wire Line
+	3800 5900 3800 5950
+Wire Wire Line
+	3800 6250 3800 6500
+Wire Wire Line
+	4300 5900 4300 5950
+Wire Wire Line
+	4300 6250 4300 6500
+Wire Wire Line
+	4800 5900 4800 5950
+Wire Wire Line
+	4800 6250 4800 6500
+Wire Wire Line
+	3300 6500 3800 6500
+$Comp
+L Mechanical:MountingHole H1
+U 1 1 5E1FD379
+P 1150 2200
+F 0 "H1" H 1250 2246 50  0000 L CNN
+F 1 "MountingHole" H 1250 2155 50  0000 L CNN
+F 2 "MountingHole:MountingHole_2.7mm" H 1150 2200 50  0001 C CNN
+F 3 "https://www.adafruit.com/product/3299" H 1150 2200 50  0001 C CNN
+	1    1150 2200
+	1    0    0    -1
+$EndComp
+$Comp
+L Mechanical:MountingHole H2
+U 1 1 5E27C5D4
+P 1150 2500
+F 0 "H2" H 1250 2546 50  0000 L CNN
+F 1 "MountingHole" H 1250 2455 50  0000 L CNN
+F 2 "MountingHole:MountingHole_2.7mm" H 1150 2500 50  0001 C CNN
+F 3 "https://www.adafruit.com/product/3299" H 1150 2500 50  0001 C CNN
+	1    1150 2500
+	1    0    0    -1
+$EndComp
+$Comp
+L Mechanical:MountingHole H3
+U 1 1 5E27C92D
+P 1150 2800
+F 0 "H3" H 1250 2846 50  0000 L CNN
+F 1 "MountingHole" H 1250 2755 50  0000 L CNN
+F 2 "MountingHole:MountingHole_2.7mm" H 1150 2800 50  0001 C CNN
+F 3 "https://www.adafruit.com/product/3299" H 1150 2800 50  0001 C CNN
+	1    1150 2800
+	1    0    0    -1
+$EndComp
+$Comp
+L Mechanical:MountingHole H4
+U 1 1 5E27CB44
+P 1150 3100
+F 0 "H4" H 1250 3146 50  0000 L CNN
+F 1 "MountingHole" H 1250 3055 50  0000 L CNN
+F 2 "MountingHole:MountingHole_2.7mm" H 1150 3100 50  0001 C CNN
+F 3 "https://www.adafruit.com/product/3299" H 1150 3100 50  0001 C CNN
+	1    1150 3100
+	1    0    0    -1
+$EndComp
+Text GLabel 11350 3150 2    39   BiDi ~ 0
+SCIB_TX
+Text GLabel 8950 3600 2    39   Output ~ 0
+Brake_PWM_1
+Text GLabel 8950 3500 2    39   Output ~ 0
+Brake_PWM_2
+Wire Wire Line
+	8100 5300 8100 5150
+Wire Wire Line
+	8200 5300 8200 5150
+Wire Wire Line
+	8300 5300 8300 5150
+Text GLabel 8950 3700 2    39   Output ~ 0
+STEERING
+Text GLabel 7900 5300 3    39   Output ~ 0
+EN+_CTL
+Text GLabel 7800 5300 3    39   Input ~ 0
+INPUT_A+_CTL
+Text GLabel 8300 5300 3    39   BiDi ~ 0
+FS1_CTL
+Text GLabel 8100 5300 3    39   BiDi ~ 0
+FWD_CTL
+Text GLabel 8000 5300 3    39   BiDi ~ 0
+REV_CTL
+Text GLabel 8200 5300 3    39   BiDi ~ 0
+KS1_CTL
+Wire Wire Line
+	8000 5150 8000 5300
+Wire Wire Line
+	7900 5150 7900 5300
+Wire Wire Line
+	7800 5150 7800 5300
+Text GLabel 5900 3750 0    39   Output ~ 0
+THROTTLE
+Wire Wire Line
+	5900 3750 6100 3750
+Wire Wire Line
+	8850 3500 8950 3500
+Wire Wire Line
+	8850 3600 8950 3600
+Wire Wire Line
+	8850 3700 8950 3700
+$Comp
+L PCB_2020:AMP_DUE_SCH U1
+U 2 1 5E636D63
+P 6400 3550
+F 0 "U1" H 6678 3496 50  0000 L CNN
+F 1 "AMP_DUE_SCH" H 6678 3405 50  0000 L CNN
+F 2 "DUE Footprint:Arduino DUE" H 6400 3550 50  0001 C CNN
+F 3 "" H 5200 4550 50  0001 C CNN
+	2    6400 3550
+	1    0    0    -1
+$EndComp
+$Comp
+L PCB_2020:AMP_DUE_SCH U1
+U 3 1 5E63B0DA
+P 8500 2500
+F 0 "U1" H 8558 2865 50  0000 C CNN
+F 1 "AMP_DUE_SCH" H 8558 2774 50  0000 C CNN
+F 2 "DUE Footprint:Arduino DUE" H 8500 2500 50  0001 C CNN
+F 3 "" H 7300 3500 50  0001 C CNN
+	3    8500 2500
+	1    0    0    -1
+$EndComp
+$Comp
+L PCB_2020:AMP_DUE_SCH U1
+U 4 1 5E63E5C9
+P 7550 4800
+F 0 "U1" H 8528 4921 50  0000 L CNN
+F 1 "AMP_DUE_SCH" H 8528 4830 50  0000 L CNN
+F 2 "DUE Footprint:Arduino DUE" H 7550 4800 50  0001 C CNN
+F 3 "" H 6350 5800 50  0001 C CNN
+	4    7550 4800
+	1    0    0    -1
+$EndComp
+NoConn ~ 6100 3550
+NoConn ~ 8850 2600
+NoConn ~ 8850 2700
+NoConn ~ 8850 2800
+NoConn ~ 8850 2900
+NoConn ~ 8850 3000
+NoConn ~ 8850 3100
+NoConn ~ 8850 3200
+NoConn ~ 8850 3300
+NoConn ~ 8850 3400
+NoConn ~ 6800 4300
+NoConn ~ 6900 4300
+NoConn ~ 7000 4300
+NoConn ~ 7100 4300
+NoConn ~ 7200 4300
+NoConn ~ 7300 4300
+NoConn ~ 7400 4300
+NoConn ~ 7500 4300
+NoConn ~ 7600 4300
+NoConn ~ 7700 4300
+NoConn ~ 7800 4300
+NoConn ~ 7900 4300
+NoConn ~ 8000 4300
+NoConn ~ 8100 4300
+NoConn ~ 8200 4300
+NoConn ~ 8300 4300
+NoConn ~ 6800 5150
+NoConn ~ 6900 5150
+NoConn ~ 7000 5150
+NoConn ~ 7100 5150
+NoConn ~ 7200 5150
+NoConn ~ 7300 5150
+NoConn ~ 7400 5150
+NoConn ~ 7500 5150
+NoConn ~ 7600 5150
+NoConn ~ 7700 5150
+$Comp
+L PCB_2020:AMP_DUE_SCH U2
+U 5 1 5E6732F5
+P 6200 2150
+F 0 "U2" H 6200 2465 50  0000 C CNN
+F 1 "AMP_DUE_SCH" H 6200 2374 50  0000 C CNN
+F 2 "DUE Footprint:Arduino DUE" H 6200 2150 50  0001 C CNN
+F 3 "" H 6750 2050 50  0001 C CNN
+	5    6200 2150
+	1    0    0    -1
+$EndComp
+$Comp
+L power:GND #GND?
+U 1 1 5E681F81
+P 6150 2700
+AR Path="/5E681F81" Ref="#GND?"  Part="1"
+AR Path="/5DF27589/5E681F81" Ref="#GND?"  Part="1"
+F 0 "#GND?" H 6150 2700 50  0001 C CNN
+F 1 "GND" H 6050 2500 59  0000 L BNN
+F 2 "" H 6150 2700 50  0001 C CNN
+F 3 "" H 6150 2700 50  0001 C CNN
+	1    6150 2700
+	1    0    0    -1
+$EndComp
+NoConn ~ 6700 2350
 $Comp
 L power:+5V #P+2
@@
 	1    0    0    -1
 $EndComp
-Text Notes 3700 7200 0    59   ~ 0
-Decoupling Caps
-$Comp
-L power:GND #GND3
-U 1 1 E2B99DEF
-P 4100 6700
-AR Path="/E2B99DEF" Ref="#GND3"  Part="1"
-AR Path="/5DF27589/E2B99DEF" Ref="#GND03"  Part="1"
-F 0 "#GND03" H 4100 6700 50  0001 C CNN
-F 1 "GND" H 4000 6500 59  0000 L BNN
-F 2 "" H 4100 6700 50  0001 C CNN
-F 3 "" H 4100 6700 50  0001 C CNN
-	1    4100 6700
-	1    0    0    -1
-$EndComp
-Wire Wire Line
-	3300 5900 3300 5950
-Wire Wire Line
-	3300 6250 3300 6500
-Wire Wire Line
-	3800 5900 3800 5950
-Wire Wire Line
-	3800 6250 3800 6500
-Wire Wire Line
-	4300 5900 4300 5950
-Wire Wire Line
-	4300 6250 4300 6500
-Wire Wire Line
-	4800 5900 4800 5950
-Wire Wire Line
-	4800 6250 4800 6500
-Wire Wire Line
-	3300 6500 3800 6500
-$Comp
-L Mechanical:MountingHole H1
-U 1 1 5E1FD379
-P 1150 2200
-F 0 "H1" H 1250 2246 50  0000 L CNN
-F 1 "MountingHole" H 1250 2155 50  0000 L CNN
-F 2 "MountingHole:MountingHole_2.7mm" H 1150 2200 50  0001 C CNN
-F 3 "https://www.adafruit.com/product/3299" H 1150 2200 50  0001 C CNN
-	1    1150 2200
-	1    0    0    -1
-$EndComp
-$Comp
-L Mechanical:MountingHole H2
-U 1 1 5E27C5D4
-P 1150 2500
-F 0 "H2" H 1250 2546 50  0000 L CNN
-F 1 "MountingHole" H 1250 2455 50  0000 L CNN
-F 2 "MountingHole:MountingHole_2.7mm" H 1150 2500 50  0001 C CNN
-F 3 "https://www.adafruit.com/product/3299" H 1150 2500 50  0001 C CNN
-	1    1150 2500
-	1    0    0    -1
-$EndComp
-$Comp
-L Mechanical:MountingHole H3
-U 1 1 5E27C92D
-P 1150 2800
-F 0 "H3" H 1250 2846 50  0000 L CNN
-F 1 "MountingHole" H 1250 2755 50  0000 L CNN
-F 2 "MountingHole:MountingHole_2.7mm" H 1150 2800 50  0001 C CNN
-F 3 "https://www.adafruit.com/product/3299" H 1150 2800 50  0001 C CNN
-	1    1150 2800
-	1    0    0    -1
-$EndComp
-$Comp
-L Mechanical:MountingHole H4
-U 1 1 5E27CB44
-P 1150 3100
-F 0 "H4" H 1250 3146 50  0000 L CNN
-F 1 "MountingHole" H 1250 3055 50  0000 L CNN
-F 2 "MountingHole:MountingHole_2.7mm" H 1150 3100 50  0001 C CNN
-F 3 "https://www.adafruit.com/product/3299" H 1150 3100 50  0001 C CNN
-	1    1150 3100
-	1    0    0    -1
-$EndComp
-Text GLabel 10100 3450 2    39   BiDi ~ 0
-SCIB_TX
-Wire Wire Line
-	10000 3450 10100 3450
-Text GLabel 10100 3250 2    39   Output ~ 0
-Brake_PWM_1
-Text GLabel 10100 3150 2    39   Output ~ 0
-Brake_PWM_2
-Wire Wire Line
-	9400 4850 9400 4700
-Wire Wire Line
-	9500 4850 9500 4700
-Wire Wire Line
-	9600 4850 9600 4700
-Text GLabel 10100 3350 2    39   Output ~ 0
-STEERING
-Text GLabel 9200 4850 3    39   Output ~ 0
-EN+_CTL
-Text GLabel 9100 4850 3    39   Input ~ 0
-INPUT_A+_CTL
-Text GLabel 9600 4850 3    39   BiDi ~ 0
-FS1_CTL
-Text GLabel 9400 4850 3    39   BiDi ~ 0
-FWD_CTL
-Text GLabel 9300 4850 3    39   BiDi ~ 0
-REV_CTL
-Text GLabel 9500 4850 3    39   BiDi ~ 0
-KS1_CTL
-Wire Wire Line
-	9300 4700 9300 4850
-Wire Wire Line
-	9200 4700 9200 4850
-Wire Wire Line
-	9100 4700 9100 4850
-Text GLabel 5900 3750 0    39   Output ~ 0
-THROTTLE
-Wire Wire Line
-	5900 3750 6100 3750
-Wire Wire Line
-	10000 3150 10100 3150
-Wire Wire Line
-	10000 3250 10100 3250
-Wire Wire Line
-	10000 3350 10100 3350
-$Comp
-L PCB_2020:AMP_DUE_SCH U1
-U 1 1 5E5CFA7A
-P 8050 3300
-F 0 "U1" H 9250 4365 50  0000 C CNN
-F 1 "AMP_DUE_SCH" H 9250 4274 50  0000 C CNN
-F 2 "DUE Footprint:Arduino DUE" H 8050 3650 50  0001 C CNN
-F 3 "" H 8050 3650 50  0001 C CNN
-	1    8050 3300
-	1    0    0    -1
+$Comp
+L power:+5V #P+?
+U 1 1 5E684B6F
+P 5700 2450
+AR Path="/5E684B6F" Ref="#P+?"  Part="1"
+AR Path="/5DF27589/5E684B6F" Ref="#P+?"  Part="1"
+F 0 "#P+?" H 5700 2450 50  0001 C CNN
+F 1 "+5V" V 5650 2550 59  0000 L BNN
+F 2 "" H 5700 2450 50  0001 C CNN
+F 3 "" H 5700 2450 50  0001 C CNN
+	1    5700 2450
+	0    -1   -1   0
+$EndComp
+$Comp
+L power:+12V #PWR?
+U 1 1 5E686230
+P 5700 2300
+F 0 "#PWR?" H 5700 2150 50  0001 C CNN
+F 1 "+12V" V 5750 2400 50  0000 L CNN
+F 2 "" H 5700 2300 50  0001 C CNN
+F 3 "" H 5700 2300 50  0001 C CNN
+	1    5700 2300
+	0    -1   -1   0
 $EndComp
 $EndSCHEMATC
